Commit message: update

File: urdf/sentinel.urdf (robot description, URDF)
Before this commit: robot mobile_robot, 6 links, 5 joints
Links:
- removed link imu_link
- link Deep_camera_link: geometry collision mesh filename=package://sentinel_bot/meshes/Deep_camera_link.STL; visual mesh filename=package://sentinel_bot/meshes/Deep_camera_link.STL
- link Left_wheel_link: geometry collision mesh filename=package://sentinel_bot/meshes/Left_wheel_link.STL; visual mesh filename=package://sentinel_bot/meshes/Left_wheel_link.STL
- link Lidar_link: geometry collision mesh filename=package://sentinel_bot/meshes/Lidar_link.STL; visual mesh filename=package://sentinel_bot/meshes/Lidar_link.STL
- link Right_wheel_link: geometry collision mesh filename=package://sentinel_bot/meshes/Right_wheel_link.STL; visual mesh filename=package://sentinel_bot/meshes/Right_wheel_link.STL
- link base_link: mass 0.321778979369154 -> 0.8; geometry collision mesh filename=package://sentinel_bot/meshes/base_link.STL; visual mesh filename=package://sentinel_bot/meshes/base_link.STL
Joints:
- removed joint imu_joint
